Commit message: bugfix urdf

File: ROS packages/rocuto_pkg/urdf/rocuto_with_macros.urdf.xacro (robot description, xacro)
@@ -58,8 +58,8 @@
     <type>transmission_interface/SimpleTransmission</type>
     <joint name="frame_to_link1">
-      <hardwareInterface>EffortJointInterface</hardwareInterface>
+      <hardwareInterface>hardware_interface/PositionJointInterface</hardwareInterface>
     </joint>
     <actuator name="link1_motor">
-      <hardwareInterface>EffortJointInterface</hardwareInterface>
+      <hardwareInterface>hardware_interface/PositionJointInterface</hardwareInterface>
       <mechanicalReduction>1</mechanicalReduction>
     </actuator>
@@ -86,8 +86,8 @@
     <type>transmission_interface/SimpleTransmission</type>
     <joint name="link1_to_link2">
-      <hardwareInterface>EffortJointInterface</hardwareInterface>
+      <hardwareInterface>hardware_interface/PositionJointInterface</hardwareInterface>
     </joint>
     <actuator name="link2_motor">
-      <hardwareInterface>EffortJointInterface</hardwareInterface>
+      <hardwareInterface>hardware_interface/PositionJointInterface</hardwareInterface>
       <mechanicalReduction>1</mechanicalReduction>
     </actuator>
@@ -119,3 +119,10 @@
     <origin xyz="${joint3_x} ${joint3_y} ${joint3_z}" rpy="0 0 0"/>
   </xacro:link_box>
+<!-- Fixed joint to make frame static in world -->
+<link name="world" />
+ <joint name="world_joint" type="fixed">
+    <parent link="world" />
+    <child link = "frame" />
+    <origin xyz="0.0 0.0 0.5" rpy="0.0 0.0 0.0" />
+ </joint>
 </robot>
