Commit message: ny

File: ROS packages/husky_simulation-main/urdf/include/husky.urdf.xacro (robot description, xacro)
@@ -57,4 +57,8 @@
   <xacro:arg name="cpr_urdf_extras" default="$(optenv CPR_URDF_EXTRAS empty.urdf)" />
   <!-- Included URDF/XACRO Files -->
+  <xacro:include filename="$(find rocuto_pkg)/urdf/rocuto_with_macros.urdf.xacro" />
+  <xacro:include filename="$(find rocuto_pkg)/urdf/macros.xacro" />
+  <xacro:include filename="$(find rocuto_pkg)/urdf/materials.xacro" />
+  <xacro:include filename="$(find rocuto_pkg)/urdf/gazebo_rocuto.urdf.gazebo" />
   <xacro:include filename="$(find husky_description)/urdf/decorations.urdf.xacro" />
   <xacro:include filename="$(find husky_description)/urdf/wheel.urdf.xacro" />

File: ROS packages/rocuto_pkg/urdf/rocuto.urdf.xacro (robot description, xacro)
@@ -66,5 +66,5 @@
     <!--<pose>0 0 0.1 0 0 0</pose> POSE ER KANSKJE IKKE NØDVENDIG-->
     <collision>
-      <origin xyz="${joint1_x} ${joint1_y} ${joint1_z}" rpy="${pi/2} 0 0"/>
+      <origin xyz="${joint1_x} ${joint1_y + 0.25} ${joint1_z}" rpy="${pi/2} 0 0"/>
       <geometry>
         <cylinder length="${link1_length}" radius="${link1_radius}"/>
@@ -72,5 +72,5 @@
     </collision>
     <visual>
-      <origin xyz="${joint1_x} ${joint1_y} ${joint1_z}" rpy="${pi/2} 0 0"/>
+      <origin xyz="${joint1_x} ${joint1_y + 0.25} ${joint1_z}" rpy="${pi/2} 0 0"/>
       <geometry>
         <cylinder length="${link1_length}" radius="${link1_radius}"/>
@@ -81,5 +81,5 @@
     <inertial>
       <mass value="1e-5" />
-<origin xyz="${joint1_x} ${joint1_y} ${joint1_z}" rpy="${pi/2} 0 0"/>
+<origin xyz="${joint1_x} ${joint1_y + 0.25} ${joint1_z}" rpy="${pi/2} 0 0"/>
       <inertia ixx="1e-6" ixy="0" ixz="0" iyy="1e-6" iyz="0" izz="1e-6" />
     </inertial>
@@ -89,5 +89,5 @@
     <!--<pose>0 0 0.1 0 0 0</pose>POSE ER KANSKJE IKKE NØDVENDIG-->
     <collision>
-      <origin xyz="${joint2_x} ${joint2_y} ${joint2_z}" rpy="${pi/2} 0 0"/>
+      <origin xyz="${joint2_x} ${joint2_y + 0.25} ${joint2_z}" rpy="${pi/2} 0 0"/>
       <geometry>
         <cylinder length="${link1_length}" radius="${link1_radius}"/>
@@ -95,5 +95,5 @@
     </collision>
     <visual>
-      <origin xyz="${joint2_x} ${joint2_y} ${joint2_z}" rpy="${pi/2} 0 0"/>
+      <origin xyz="${joint2_x} ${joint2_y + 0.25} ${joint2_z}" rpy="${pi/2} 0 0"/>
       <geometry>
         <cylinder length="${link1_length}" radius="${link1_radius}"/>
@@ -104,5 +104,5 @@
     <inertial>
       <mass value="1e-5" />
-      <origin xyz="${joint2_x} ${joint2_y} ${joint2_z}" rpy="${pi/2} 0 0"/>
+      <origin xyz="${joint2_x} ${joint2_y + 0.25} ${joint2_z}" rpy="${pi/2} 0 0"/>
       <inertia ixx="1e-6" ixy="0" ixz="0" iyy="1e-6" iyz="0" izz="1e-6" />
     </inertial>
@@ -112,5 +112,5 @@
     <!--<pose>0 0 0.1 0 0 0</pose>POSE ER KANSKJE IKKE NØDVENDIG-->
     <collision>
-      <origin xyz="${joint3_x} ${joint3_y} ${joint3_z}" rpy="0 0 0"/>
+      <origin xyz="${joint3_x} ${joint3_y + 0.25} ${joint3_z}" rpy="0 0 0"/>
       <geometry>
         <box size="${tool_length} ${tool_width} ${tool_height}"/>
@@ -118,5 +118,5 @@
     </collision>
     <visual>
-      <origin xyz="${joint3_x} ${joint3_y} ${joint3_z}" rpy="0 0 0"/>
+      <origin xyz="${joint3_x} ${joint3_y + 0.25} ${joint3_z}" rpy="0 0 0"/>
       <geometry>
         <box size="${tool_length} ${tool_width} ${tool_height}"/>
@@ -127,5 +127,5 @@
     <inertial>
       <mass value="1e-5" />
-      <origin xyz="${joint3_x} ${joint3_y} ${joint3_z}" rpy="0 0 0"/>
+      <origin xyz="${joint3_x} ${joint3_y + 0.25} ${joint3_z}" rpy="0 0 0"/>
       <inertia ixx="1e-6" ixy="0" ixz="0" iyy="1e-6" iyz="0" izz="1e-6" />
     </inertial>

File: ROS packages/rocuto_pkg/urdf/rocuto_with_macros.urdf.xacro (robot description, xacro)
@@ -7,4 +7,8 @@
   <!-- constants -->
   <xacro:property name="M_PI" value="3.14159"/>
+  <!-- world properties -->
+  <xacro:property name="world_x" value="0.0" />
+  <xacro:property name="world_y" value="0.0" />
+  <xacro:property name="world_z" value="0.5" />
   <!-- frame properties -->
   <xacro:property name="frame_x_size" value="0.2" />
@@ -24,25 +28,41 @@
   <xacro:property name="frame_x_origin" value="0" />
   <xacro:property name="frame_y_origin" value="0" />
-  <xacro:property name="frame_z_origin" value="0.5" />
+  <xacro:property name="frame_z_origin" value="0.05" />
   <!-- joint 1 origin -->
-  <xacro:property name="joint1_x" value="${frame_x_origin}" />
-  <xacro:property name="joint1_y" value="${frame_y_origin + 0.2}" />
-  <xacro:property name="joint1_z" value="${frame_z_origin - 0.5}" />
+  <xacro:property name="joint1_x" value="0" />
+  <xacro:property name="joint1_y" value="${frame_y_size}" />
+  <xacro:property name="joint1_z" value="0" />
   <!-- joint 2 origin -->
-  <xacro:property name="joint2_x" value="${frame_x_origin}" />
-  <xacro:property name="joint2_y" value="${frame_y_origin + 0.2 + 0.5}" />
-  <xacro:property name="joint2_z" value="${frame_z_origin - 0.5}" />
+  <xacro:property name="joint2_x" value="0" />
+  <xacro:property name="joint2_y" value="${link1_length}" />
+  <xacro:property name="joint2_z" value="0" />
   <!-- joint 3 origin -->
-  <xacro:property name="joint3_x" value="${frame_x_origin}" />
-  <xacro:property name="joint3_y" value="${frame_y_origin + 0.2 + 0.5 + 0.5}" />
-  <xacro:property name="joint3_z" value="${frame_z_origin - 0.5}" />
+  <xacro:property name="joint3_x" value="0" />
+  <xacro:property name="joint3_y" value="${link1_length}" />
+  <xacro:property name="joint3_z" value="0" />
+  <!-- frame visual/collision/inertial origin -->
+  <xacro:property name="frame_x_vis" value="${frame_x_origin}" />
+  <xacro:property name="frame_y_vis" value="${frame_y_origin}" />
+  <xacro:property name="frame_z_vis" value="${frame_z_origin}" />
+  <!-- link 1 visual/collision/inertial origin -->
+  <xacro:property name="link1_x_vis" value="${joint1_x}" />
+  <xacro:property name="link1_y_vis" value="${joint1_y}" />
+  <xacro:property name="link1_z_vis" value="${joint1_z}" />
+  <!-- link 2 visual/collision/inertial origin -->
+  <xacro:property name="link2_x_vis" value="${joint2_x}" />
+  <xacro:property name="link2_y_vis" value="${joint2_y}" />
+  <xacro:property name="link2_z_vis" value="${joint2_z}" />
+  <!-- tool visual/collision/inertial origin -->
+  <xacro:property name="tool_x_vis" value="${joint3_x - 0.05}" />
+  <xacro:property name="tool_y_vis" value="${joint3_y + 0.25}" />
+  <xacro:property name="tool_z_vis" value="${joint3_z - 0.05}" />
 <!-- ramme på robotplatform -->
   <xacro:link_box link_name="frame" length="${frame_x_size}" width="${frame_y_size}" height="${frame_z_size}" density="1" mesh_name="nofile">
     <!-- origin visual -->
-    <origin xyz="${frame_x_origin} ${frame_y_origin} ${frame_z_origin}" rpy="0 0 0"/>
+    <origin xyz="${frame_x_vis} ${frame_y_vis} ${frame_z_vis}" rpy="0 0 0"/>
     <!-- origin collision -->
-    <origin xyz="${frame_x_origin} ${frame_y_origin} ${frame_z_origin}" rpy="0 0 0"/>
+    <origin xyz="${frame_x_vis} ${frame_y_vis} ${frame_z_vis}" rpy="0 0 0"/>
     <!-- origin inertia -->
-    <origin xyz="${frame_x_origin} ${frame_y_origin} ${frame_z_origin}" rpy="0 0 0"/>
+    <origin xyz="${frame_x_vis} ${frame_y_vis} ${frame_z_vis}" rpy="0 0 0"/>
   </xacro:link_box>
   <!-- leddet mellom ramme og link1 -->
@@ -68,9 +88,9 @@
   <xacro:link_cylinder link_name="link1" radius="${link1_radius}" length="${link1_length}" density="1" mesh_name="nofile">
     <!-- origin visual -->
-    <origin xyz="${joint1_x} ${joint1_y + 0.25} ${joint1_z}" rpy="${M_PI/2} 0 0"/>
+    <origin xyz="${link1_x_vis} ${link1_y_vis} ${link1_z_vis}" rpy="${M_PI/2} 0 0"/>
     <!-- origin collision -->
-    <origin xyz="${joint1_x} ${joint1_y + 0.25} ${joint1_z}" rpy="${M_PI/2} 0 0"/>
+    <origin xyz="${link1_x_vis} ${link1_y_vis} ${link1_z_vis}" rpy="${M_PI/2} 0 0"/>
     <!-- origin inertia -->
-    <origin xyz="${joint1_x} ${joint1_y} ${joint1_z}" rpy="${M_PI/2} 0 0"/>
+    <origin xyz="${link1_x_vis} ${link1_y_vis} ${link1_z_vis}" rpy="${M_PI/2} 0 0"/>
   </xacro:link_cylinder>
   <!-- leddet mellom link1 og link2 -->
@@ -80,5 +100,5 @@
     <child link="link2"/>
     <axis xyz="0 0 1" rpy="0 0 0"/>
-    <limit effort="100" velocity="100" lower="-${pi/2}" upper="${pi/2}"/>
+    <limit effort="100" velocity="100" lower="-${3*pi/4}" upper="${3*pi/4}"/>
     <joint_properties damping="0.0" friction="0.0"/>
   </joint>
@@ -95,9 +115,10 @@
 <!-- link2 -->
   <xacro:link_cylinder link_name="link2" radius="${link1_radius}" length="${link1_length}" density="1" mesh_name="nofile">
-    <origin xyz="${joint2_x} ${joint2_y + 0.25} ${joint2_z}" rpy="${M_PI/2} 0 0"/>
+    <!-- origin visual -->
+    <origin xyz="${link2_x_vis} ${link2_y_vis} ${link2_z_vis}" rpy="${M_PI/2} 0 0"/>
     <!-- origin collision -->
-    <origin xyz="${joint2_x} ${joint2_y + 0.25} ${joint2_z}" rpy="${M_PI/2} 0 0"/>
+    <origin xyz="${link2_x_vis} ${link2_y_vis} ${link2_z_vis}" rpy="${M_PI/2} 0 0"/>
     <!-- origin inertia -->
-    <origin xyz="${joint2_x} ${joint2_y} ${joint2_z}" rpy="${M_PI/2} 0 0"/>
+    <origin xyz="${link2_x_vis} ${link2_y_vis} ${link2_z_vis}" rpy="${M_PI/2} 0 0"/>
   </xacro:link_cylinder>
 <!-- Dette er ikke et ledd bare kobling mellom link2 og tool -->
@@ -113,9 +134,9 @@
   <xacro:link_box link_name="tool" length="${tool_length}" width="${tool_width}" height="${tool_height}" density="1" mesh_name="nofile">
     <!-- origin visual -->
-    <origin xyz="${joint3_x} ${joint3_y} ${joint3_z}" rpy="0 0 0"/>
+    <origin xyz="${tool_x_vis} ${tool_y_vis} ${tool_z_vis}" rpy="0 0 0"/>
     <!-- origin collision -->
-    <origin xyz="${joint3_x} ${joint3_y} ${joint3_z}" rpy="0 0 0"/>
+    <origin xyz="${tool_x_vis} ${tool_y_vis} ${tool_z_vis}" rpy="0 0 0"/>
     <!-- origin inertia -->
-    <origin xyz="${joint3_x} ${joint3_y} ${joint3_z}" rpy="0 0 0"/>
+    <origin xyz="${tool_x_vis} ${tool_y_vis} ${tool_z_vis}" rpy="0 0 0"/>
   </xacro:link_box>
 <!-- Fixed joint to make frame static in world -->
@@ -124,5 +145,5 @@
     <parent link="world" />
     <child link = "frame" />
-    <origin xyz="0.0 0.0 0.5" rpy="0.0 0.0 0.0" />
+    <origin xyz="${world_x} ${world_y} ${world_z}" rpy="0.0 0.0 0.0" />
  </joint>
 </robot>

Commit message: ny

File: ROS packages/husky_simulation-main/urdf/include/husky.urdf.xacro (robot description, xacro)
@@ -121,4 +121,9 @@
     <child link="inertial_link" />
   </joint>
+  <joint name="rocuto_joint" type="fixed">
+    <origin xyz="0 0.5708 0" rpy="0 0 0" />
+    <parent link="base_link" />
+    <child link="frame" />
+  </joint>
   <!-- IMU Link is the standard mounting position for the UM6 IMU.-->
   <!-- Can be modified with environment variables in /etc/ros/setup.bash 0 -1.5708 3.1416-->
